File: PCB/laser-tag-sao.kicad_sch (KiCad schematic)
At the start: 0 parts

Commit message: almost done schematic!
Parts:
- added BZ1: Buzzer, symbol Device:Buzzer
- added C1: 10uF, symbol Device:C
- added D1: VSLY5940, symbol Device:D
- added D2, D3, D4: WS2812B-4020, WS2812B-4020:LED_WS2812B-4020, symbol kai-library:WS2812B-4020
- added J1: SAO Connector, symbol Connector_Generic:Conn_02x03_Odd_Even
- added Q1: PN2222A, Package_TO_SOT_THT:TO-92_Inline, symbol Transistor_BJT:PN2222A
- added R1: 22, symbol Device:R
- added R2: 1k, symbol Device:R
- added R3: 100, symbol Device:R
- added U1: ATtiny84-20P, Package_DIP:DIP-14_W7.62mm, symbol MCU_Microchip_ATtiny:ATtiny84-20P
- added U2: TSOP38438, OptoDevice:Vishay_MINICAST-3Pin, symbol Interface_Optical:TSOP384xx
- added U3: OLED_0.91_128x32, Hackclub Footprints:OLED_0.91_128x32, symbol Hackclub Symbols:OLED_0.91_128x32
Connections:
- new net: D3.3 (DOUT), D4.1 (DIN)
- new net: Q1.2 (B), R2.2
- new net: R3.2, U2.3 (Vs)
- new net: D1.1 (K), Q1.3 (C)
- new net: D1.2 (A), R1.2
- new net: D2.3 (DOUT), D3.1 (DIN)
- new net +3V3: C1.1, D2.2 (VDD), D3.2 (VDD), D4.2 (VDD), J1.1 (Pin_1), R1.1, R3.1, U1.1 (VCC), U3.2 (VCC)
- new net BUZZER: BZ1.1 (+), U1.2 (XTAL1/PB0)
- new net GND: BZ1.2 (-), C1.2, D2.4 (VSS), D3.4 (VSS), D4.4 (VSS), J1.2 (Pin_2), Q1.1 (E), U1.14 (GND), U2.2 (GND), U3.1 (GND)
- new net IR_RX: U1.5 (PB2), U2.1 (OUT)
- new net LED: D2.1 (DIN), U1.6 (PA7)
- new net MISO/IR_TX: J1.5 (Pin_5), R2.1, U1.8 (PA5)
- new net MOSI/SDA: J1.3 (Pin_3), U1.7 (PA6)
- new net OLED_SCL: U1.12 (PA1), U3.3 (SCL)
- new net OLED_SDA: U1.13 (AREF/PA0), U3.4 (SDA)
- new net RESET: J1.6 (Pin_6), U1.4 (~{RESET}/PB3)
- new net SCK/SCL: J1.4 (Pin_4), U1.9 (PA4)
- no-connect marks 0 -> 1
Other:
- note added: "SAO connector for both programming and I2C"
- note added: "Singular MCC for decoupling for the whole board"

Commit message: finished schematic
Parts:
- added R4: R, symbol Device:R
- added SW1, SW2, SW3: SW_Push, symbol Switch:SW_Push
Connections:
- net +3V3: now also R4.1
- net GND: now also SW1.2, SW2.2, SW3.2
- net RESET: now also R4.2
- net PUSH2: now reaches U1.10 (PA3)
- net PUSH2: now also SW2.1
- net PUSH1: now reaches U1.11 (PA2)
- net PUSH1: now also SW1.1
- net PUSH3: now reaches U1.3 (XTAL2/PB1)
- net PUSH3: now also SW3.1
Other:
- moved on the sheet: C1

Commit message: updating schematic again
Parts:
- added JP1, JP2: Bridged Jumper, symbol Jumper:SolderJumper_2_Bridged
- R4: value R -> 10k
Connections:
- net MISO/IR_TX: now also JP1.1 (A); no longer J1.5 (Pin_5)
- net RESET: now also JP2.2 (B); no longer J1.6 (Pin_6)
- new net: J1.5 (Pin_5), JP1.2 (B)
- new net: J1.6 (Pin_6), JP2.1 (A)
Other:
- moved on the sheet: J1

Commit message: updating again
Parts:
- removed R3: 100, symbol Device:R
Connections:
- net +3V3: now also U2.3 (Vs)
Other:
- moved on the sheet: U2
Changed lines of the file:
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@@
-	(wire
-		(pts
-			(xy 223.52 33.02) (xy 227.33 33.02)
-		)
-		(stroke
-			(width 0)
-			(type default)
-		)
-	)
 	(wire
 		(pts
@@
 	(wire
 		(pts
-			(xy 223.52 38.1) (xy 237.49 38.1)
+			(xy 222.25 38.1) (xy 236.22 38.1)
 		)
 		(stroke
@@
 	(wire
 		(pts
+			(xy 234.95 30.48) (xy 234.95 33.02)
+		)
+		(stroke
+			(width 0)
+			(type default)
+		)
+	)
+	(wire
+		(pts
 			(xy 157.48 46.99) (xy 144.78 46.99)
 		)
@@
 	(wire
 		(pts
-			(xy 236.22 43.18) (xy 236.22 45.72)
+			(xy 234.95 43.18) (xy 234.95 45.72)
 		)
 		(stroke
@@
 	(wire
 		(pts
+			(xy 234.95 33.02) (xy 236.22 33.02)
+		)
+		(stroke
+			(width 0)
+			(type default)
+		)
+	)
+	(wire
+		(pts
 			(xy 30.48 41.91) (xy 44.45 41.91)
 		)
@@
 	(wire
 		(pts
-			(xy 237.49 43.18) (xy 236.22 43.18)
+			(xy 236.22 43.18) (xy 234.95 43.18)
 		)
 		(stroke
@@
 		(pts
 			(xy 167.64 74.93) (xy 144.78 74.93)
-		)
-		(stroke
-			(width 0)
-			(type default)
-		)
-	)
-	(wire
-		(pts
-			(xy 234.95 33.02) (xy 237.49 33.02)
 		)
 		(stroke
@@
 	)
 	(label "IR_RX"
-		(at 223.52 38.1 0)
+		(at 222.25 38.1 0)
 		(effects
 			(font
@@
 	(symbol
 		(lib_id "power:+3V3")
-		(at 223.52 33.02 0)
+		(at 234.95 30.48 0)
 		(unit 1)
 		(body_style 1)
@@
 		(fields_autoplaced yes)
 		(property "Reference" "#PWR017"
-			(at 223.52 36.83 0)
+			(at 234.95 34.29 0)
 			(hide yes)
 			(show_name no)
@@
 		)
 		(property "Value" "+3V3"
-			(at 223.52 27.94 0)
+			(at 234.95 25.4 0)
 			(show_name no)
 			(do_not_autoplace no)
@@
 		)
 		(property "Footprint" ""
-			(at 223.52 33.02 0)
+			(at 234.95 30.48 0)
 			(hide yes)
 			(show_name no)
@@
 		)
 		(property "Datasheet" ""
-			(at 223.52 33.02 0)
+			(at 234.95 30.48 0)
 			(hide yes)
 			(show_name no)
@@
 		)
 		(property "Description" "Power symbol creates a global label with name \"+3V3\""
-			(at 223.52 33.02 0)
+			(at 234.95 30.48 0)
 			(hide yes)
 			(show_name no)
@@
 				(path "/bd497134-ab55-4d01-915d-3710c30e2e14"
 					(reference "#PWR017")
-					(unit 1)
-				)
-			)
-		)
-	)
-	(symbol
-		(lib_id "Device:R")
-		(at 231.14 33.02 90)
-		(unit 1)
-		(body_style 1)
-		(exclude_from_sim no)
-		(in_bom yes)
-		(on_board yes)
-		(in_pos_files yes)
-		(dnp no)
-		(fields_autoplaced yes)
-		(property "Reference" "R3"
-			(at 231.14 26.67 90)
-			(show_name no)
-			(do_not_autoplace no)
-			(effects
-				(font
-					(size 1.27 1.27)
-				)
-			)
-		)
-		(property "Value" "100"
-			(at 231.14 29.21 90)
-			(show_name no)
-			(do_not_autoplace no)
-			(effects
-				(font
-					(size 1.27 1.27)
-				)
-			)
-		)
-		(property "Footprint" ""
-			(at 231.14 34.798 90)
-			(hide yes)
-			(show_name no)
-			(do_not_autoplace no)
-			(effects
-				(font
-					(size 1.27 1.27)
-				)
-			)
-		)
-		(property "Datasheet" ""
-			(at 231.14 33.02 0)
-			(hide yes)
-			(show_name no)
-			(do_not_autoplace no)
-			(effects
-				(font
-					(size 1.27 1.27)
-				)
-			)
-		)
-		(property "Description" "Resistor"
-			(at 231.14 33.02 0)
-			(hide yes)
-			(show_name no)
-			(do_not_autoplace no)
-			(effects
-				(font
-					(size 1.27 1.27)
-				)
-			)
-		)
-		(pin "2"
-		)
-		(pin "1"
-		)
-		(instances
-			(project "laser-tag-sao"
-				(path "/bd497134-ab55-4d01-915d-3710c30e2e14"
-					(reference "R3")
 					(unit 1)
 				)
@@
 	(symbol
 		(lib_id "Interface_Optical:TSOP384xx")
-		(at 247.65 38.1 0)
+		(at 246.38 38.1 0)
 		(mirror y)
 		(unit 1)
@@
 		(dnp no)
 		(property "Reference" "U2"
-			(at 260.35 39.3701 0)
+			(at 259.08 39.3701 0)
 			(show_name no)
 			(do_not_autoplace no)
@@
 		)
 		(property "Value" "TSOP38438"
-			(at 260.35 36.8301 0)
+			(at 259.08 36.8301 0)
 			(show_name no)
 			(do_not_autoplace no)
@@
 		)
 		(property "Footprint" "OptoDevice:Vishay_MINICAST-3Pin"
-			(at 248.92 47.625 0)
+			(at 247.65 47.625 0)
 			(hide yes)
 			(show_name no)
@@
 		)
 		(property "Datasheet" "http://www.vishay.com/docs/82491/tsop382.pdf"
-			(at 231.14 30.48 0)
+			(at 229.87 30.48 0)
 			(hide yes)
 			(show_name no)
@@
 		)
 		(property "Description" "Photo Modules for PCM Remote Control Systems"
-			(at 247.65 38.1 0)
+			(at 246.38 38.1 0)
 			(hide yes)
 			(show_name no)
@@
 	(symbol
 		(lib_id "power:GND")
-		(at 236.22 45.72 0)
+		(at 234.95 45.72 0)
 		(unit 1)
 		(body_style 1)
@@
 		(fields_autoplaced yes)
 		(property "Reference" "#PWR07"
-			(at 236.22 52.07 0)
+			(at 234.95 52.07 0)
 			(hide yes)
 			(show_name no)
@@
 		)
 		(property "Value" "GND"
-			(at 236.22 50.8 0)
+			(at 234.95 50.8 0)
 			(show_name no)
 			(do_not_autoplace no)
@@
 		)
 		(property "Footprint" ""
-			(at 236.22 45.72 0)
+			(at 234.95 45.72 0)
 			(hide yes)
 			(show_name no)
@@
 		)
 		(property "Datasheet" ""
-			(at 236.22 45.72 0)
+			(at 234.95 45.72 0)
 			(hide yes)
 			(show_name no)
@@
 		)
 		(property "Description" "Power symbol creates a global label with name \"GND\" , ground"
-			(at 236.22 45.72 0)
-			(hide yes)
-			(show_name no)
+			(at 234.95 45.72 0)
+			(hide yes)
+			(show_name no)

Commit message: adding in some part #s
Parts:
- D1: Digikey Part # (none) -> VSLY5940-ND
- U1: value ATtiny84-20P -> ATTINY84A-PU; Digikey Part # (none) -> ATTINY84A-PU-ND
- U2: Digikey Part # (none) -> TSOP38438-ND
Other:
- note added: "Singular MLCC for decoupling for the whole board"
- note removed: "Singular MCC for decoupling for the whole board"
Changed lines of the file:
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@@
 		)
 	)
-	(text "Singular MCC for decoupling \nfor the whole board"
+	(text "Singular MLCC for decoupling \nfor the whole board"
 		(exclude_from_sim no)
 		(at 179.832 29.972 0)
@@
 			)
 		)
+		(property "Digikey Part #" "VSLY5940-ND"
+			(at 250.19 80.01 90)
+			(hide yes)
+			(show_name no)
+			(do_not_autoplace no)
+			(effects
+				(font
+					(size 1.27 1.27)
+				)
+			)
+		)
 		(pin "2"
 		)
@@
 			)
 		)
+		(property "Digikey Part #" "TSOP38438-ND"
+			(at 246.38 38.1 0)
+			(hide yes)
+			(show_name no)
+			(do_not_autoplace no)
+			(effects
+				(font
+					(size 1.27 1.27)
+				)
+			)
+		)
 		(pin "1"
 		)
@@
 			)
 		)
-		(property "Value" "ATtiny84-20P"
+		(property "Value" "ATTINY84A-PU"
 			(at 115.57 60.9599 0)
 			(show_name no)
@@
 			(at 129.54 59.69 0)
 			(hide yes)
+			(show_name no)
+			(do_not_autoplace no)
+			(effects
+				(font
+					(size 1.27 1.27)
+				)
+			)
+		)
+		(property "Digikey Part #" "ATTINY84A-PU-ND"
+			(at 129.54 59.69 0)
+			(hide yes)

Commit message: adding in all the footprints
Parts:
- removed JP1, JP2: Bridged Jumper, symbol Jumper:SolderJumper_2_Bridged
- added JP1, JP2: Jumper_2_Open, Jumper:SolderJumper-2_P1.3mm_Open_RoundedPad1.0x1.5mm, symbol Jumper:Jumper_2_Open
- BZ1: footprint (none) -> Buzzer_Beeper:Buzzer_TDK_PS1240P02BT_D12.2mm_H6.5mm; Digikey Part # (none) -> 445-2525-1-ND - Cut Tape (CT)
- C1: footprint (none) -> Capacitor_THT:C_Disc_D5.0mm_W2.5mm_P2.50mm; Digikey Part # (none) -> 445-173132-1-ND - Cut Tape (CT)
- D1: footprint (none) -> LED_THT:LED_D5.0mm
- J1: footprint (none) -> Connector_PinHeader_2.54mm:PinHeader_2x03_P2.54mm_Vertical
- R1: footprint (none) -> Resistor_THT:R_Axial_DIN0309_L9.0mm_D3.2mm_P12.70mm_Horizontal; Digikey Part # (none) -> 445-173132-1-ND - Cut Tape (CT)
- R2: footprint (none) -> Resistor_THT:R_Axial_DIN0309_L9.0mm_D3.2mm_P12.70mm_Horizontal; Digikey Part # (none) -> CF12JT1K00TR-ND - Tape & Reel (TR)
- R4: footprint (none) -> Resistor_THT:R_Axial_DIN0309_L9.0mm_D3.2mm_P12.70mm_Horizontal; Digikey Part # (none) -> CF12JT10K0TR-ND - Tape & Reel (TR)
- SW1: footprint (none) -> Button_Switch_THT:SW_PUSH_6mm; Digikey Part # (none) -> 450-1650-ND
- SW2, SW3: footprint (none) -> Button_Switch_THT:SW_PUSH_6mm
Connections:
- net MISO/IR_TX: now also JP1.1 (A)
- net RESET: now also JP2.2 (B)
- net at J1.5 (Pin_5): now also JP1.2 (B)
- net at J1.6 (Pin_6): now also JP2.1 (A)
Other:
- title: (none) -> Laser Tag SAOs

Commit message: laying out components on my board
Parts:
- R1: footprint Resistor_THT:R_Axial_DIN0309_L9.0mm_D3.2mm_P12.70mm_Horizontal -> Resistor_THT:R_Axial_DIN0204_L3.6mm_D1.6mm_P5.08mm_Horizontal; Digikey Part # 445-173132-1-ND - Cut Tape (CT) -> CF18JT22R0TR-ND - Tape & Reel (TR)
- R2: footprint Resistor_THT:R_Axial_DIN0309_L9.0mm_D3.2mm_P12.70mm_Horizontal -> Resistor_THT:R_Axial_DIN0204_L3.6mm_D1.6mm_P5.08mm_Horizontal; Digikey Part # CF12JT1K00TR-ND - Tape & Reel (TR) -> CF18JT1K00TR-ND - Tape & Reel (TR)
- R4: footprint Resistor_THT:R_Axial_DIN0309_L9.0mm_D3.2mm_P12.70mm_Horizontal -> Resistor_THT:R_Axial_DIN0204_L3.6mm_D1.6mm_P5.08mm_Horizontal; Digikey Part # CF12JT10K0TR-ND - Tape & Reel (TR) -> CF18JT10K0TR-ND - Tape & Reel (TR)
Changed lines of the file:
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@@
 			)
 		)
-		(property "Footprint" "Resistor_THT:R_Axial_DIN0309_L9.0mm_D3.2mm_P12.70mm_Horizontal"
+		(property "Footprint" "Resistor_THT:R_Axial_DIN0204_L3.6mm_D1.6mm_P5.08mm_Horizontal"
 			(at 165.862 68.58 90)
 			(hide yes)
@@
 			)
 		)
-		(property "Digikey Part #" "CF12JT10K0TR-ND - Tape & Reel (TR)"
+		(property "Digikey Part #" "CF18JT10K0TR-ND - Tape & Reel (TR)"
 			(at 167.64 68.58 0)
 			(hide yes)
@@
 			)
 		)
-		(property "Footprint" "Resistor_THT:R_Axial_DIN0309_L9.0mm_D3.2mm_P12.70mm_Horizontal"
+		(property "Footprint" "Resistor_THT:R_Axial_DIN0204_L3.6mm_D1.6mm_P5.08mm_Horizontal"
 			(at 236.22 93.218 90)
 			(hide yes)
@@
 			)
 		)
-		(property "Digikey Part #" "CF12JT1K00TR-ND - Tape & Reel (TR)"
+		(property "Digikey Part #" "CF18JT1K00TR-ND - Tape & Reel (TR)"
 			(at 236.22 91.44 90)
 			(hide yes)
@@
 			)
 		)
-		(property "Footprint" "Resistor_THT:R_Axial_DIN0309_L9.0mm_D3.2mm_P12.70mm_Horizontal"
+		(property "Footprint" "Resistor_THT:R_Axial_DIN0204_L3.6mm_D1.6mm_P5.08mm_Horizontal"
 			(at 248.412 69.85 90)
 			(hide yes)
@@
 			)
 		)
-		(property "Digikey Part #" "445-173132-1-ND - Cut Tape (CT)"
+		(property "Digikey Part #" "CF18JT22R0TR-ND - Tape & Reel (TR)"
 			(at 250.19 69.85 0)
 			(hide yes)

Commit message: adding neopixels and soldermask openings
Parts:
- removed SW3: SW_Push, Button_Switch_THT:SW_PUSH_6mm, symbol Switch:SW_Push
- D2, D3, D4: footprint WS2812B-4020:LED_WS2812B-4020 -> kai's library:LED_WS2812B-4020
Changed lines of the file:
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@@
 		(exclude_from_sim no)
 		(at 208.28 118.11 0)
-		(size 69.85 45.72)
+		(size 69.85 38.1)
 		(margins 0.9525 0.9525 0.9525 0.9525)
 		(stroke
@@
 	)
 	(junction
-		(at 264.16 153.67)
-		(diameter 0)
-		(color 0 0 0 0)
-	)
-	(junction
 		(at 143.51 134.62)
 		(diameter 0)
@@
 	(wire
 		(pts
-			(xy 264.16 153.67) (xy 264.16 156.21)
+			(xy 264.16 140.97) (xy 264.16 146.05)
 		)
 		(stroke
@@
 	(wire
 		(pts
-			(xy 264.16 140.97) (xy 264.16 153.67)
-		)
-		(stroke
-			(width 0)
-			(type default)
-		)
-	)
-	(wire
-		(pts
 			(xy 113.03 134.62) (xy 143.51 134.62)
 		)
@@
 	(wire
 		(pts
-			(xy 248.92 153.67) (xy 264.16 153.67)
-		)
-		(stroke
-			(width 0)
-			(type default)
-		)
-	)
-	(wire
-		(pts
 			(xy 67.31 44.45) (xy 57.15 44.45)
 		)
@@
 	(wire
 		(pts
-			(xy 238.76 153.67) (xy 224.79 153.67)
-		)
-		(stroke
-			(width 0)
-			(type default)
-		)
-	)
-	(wire
-		(pts
 			(xy 144.78 59.69) (xy 157.48 59.69)
 		)
@@
 		)
 	)
-	(label "PUSH3"
-		(at 224.79 153.67 0)
-		(effects
-			(font
-				(size 1.27 1.27)
-			)
-			(justify left bottom)
-		)
-	)
 	(label "OLED_SDA"
 		(at 157.48 44.45 180)
@@
 	)
 	(symbol
-		(lib_id "Switch:SW_Push")
-		(at 243.84 153.67 0)
-		(unit 1)
-		(body_style 1)
-		(exclude_from_sim no)
-		(in_bom yes)
-		(on_board yes)
-		(in_pos_files yes)
-		(dnp no)
-		(fields_autoplaced yes)
-		(property "Reference" "SW3"
-			(at 243.84 146.05 0)
-			(show_name no)
-			(do_not_autoplace no)
-			(effects
-				(font
-					(size 1.27 1.27)
-				)
-			)
-		)
-		(property "Value" "SW_Push"
-			(at 243.84 148.59 0)
-			(show_name no)
-			(do_not_autoplace no)
-			(effects
-				(font
-					(size 1.27 1.27)
-				)
-			)
-		)
-		(property "Footprint" "Button_Switch_THT:SW_PUSH_6mm"
-			(at 243.84 148.59 0)
-			(hide yes)
-			(show_name no)
-			(do_not_autoplace no)
-			(effects
-				(font
-					(size 1.27 1.27)
-				)
-			)
-		)
-		(property "Datasheet" ""
-			(at 243.84 148.59 0)
-			(hide yes)
-			(show_name no)
-			(do_not_autoplace no)
-			(effects
-				(font
-					(size 1.27 1.27)
-				)
-			)
-		)
-		(property "Description" "Push button switch, generic, two pins"
-			(at 243.84 153.67 0)
-			(hide yes)
-			(show_name no)
-			(do_not_autoplace no)
-			(effects
-				(font
-					(size 1.27 1.27)
-				)
-			)
-		)
-		(pin "1"
-		)
-		(pin "2"
-		)
-		(instances
-			(project "laser-tag-sao"
-				(path "/bd497134-ab55-4d01-915d-3710c30e2e14"
-					(reference "SW3")
-					(unit 1)
-				)
-			)
-		)
-	)
-	(symbol
 		(lib_id "power:+3V3")
 		(at 54.61 106.68 0)
@@
 			)
 		)
-		(property "Footprint" "WS2812B-4020:LED_WS2812B-4020"
+		(property "Footprint" "kai's library:LED_WS2812B-4020"
 			(at 173.99 124.46 0)
 			(hide yes)
@@
 	(symbol
 		(lib_id "power:GND")
-		(at 264.16 156.21 0)
+		(at 264.16 146.05 0)
 		(unit 1)
 		(body_style 1)
@@
 		(fields_autoplaced yes)
 		(property "Reference" "#PWR01"
-			(at 264.16 162.56 0)
+			(at 264.16 152.4 0)
 			(hide yes)
 			(show_name no)
@@
 		)
 		(property "Value" "GND"
-			(at 264.16 161.29 0)
+			(at 264.16 151.13 0)
 			(show_name no)
 			(do_not_autoplace no)
@@
 		)
 		(property "Footprint" ""
-			(at 264.16 156.21 0)
+			(at 264.16 146.05 0)
 			(hide yes)
 			(show_name no)
@@
 		)
 		(property "Datasheet" ""
-			(at 264.16 156.21 0)
+			(at 264.16 146.05 0)
 			(hide yes)
 			(show_name no)
@@
 		)
 		(property "Description" "Power symbol creates a global label with name \"GND\" , ground"
-			(at 264.16 156.21 0)
+			(at 264.16 146.05 0)
 			(hide yes)
 			(show_name no)
@@
 			)
 		)
-		(property "Footprint" "WS2812B-4020:LED_WS2812B-4020"
+		(property "Footprint" "kai's library:LED_WS2812B-4020"
 			(at 143.51 124.46 0)
 			(hide yes)
@@
 			)
 		)
-		(property "Footprint" "WS2812B-4020:LED_WS2812B-4020"
+		(property "Footprint" "kai's library:LED_WS2812B-4020"
 			(at 113.03 124.46 0)
 			(hide yes)
