File: PCB/laser-tag-sao.kicad_sch (KiCad schematic)
At the start: 18 parts, among them J1 SAO Connector, Q1 PN2222A, SW1 SW_Push, SW2 SW_Push, U1 ATTINY84A-PU, U2 TSOP38438, U3 OLED_0.91_128x32

Commit message: finished routing the board, 0 DRC errors
Connections:
- net PUSH3 is gone; now on net PUSH2: U1.3 (XTAL2/PB1)
- net PUSH2: no longer U1.10 (PA3)
- no-connect marks 1 -> 2

Commit message: new digikey BOM
Parts:
- J1: Digikey Part # (none) -> 35-PRPC003DAAN-RC-ND
Changed lines of the file:
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@@
+			)
+		)
+		(property "Digikey Part #" "35-PRPC003DAAN-RC-ND"
+			(at 49.53 44.45 0)
+			(hide yes)
+			(show_name no)
+			(do_not_autoplace no)
+			(effects
+				(font
+					(size 1.27 1.27)
+				)
 			)
 		)

Commit message: updating BOM
Parts:
- Q1: Digikey Part # (none) -> 1514-PN2222APBFREE-ND
Changed lines of the file:
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@@
+			)
+		)
+		(property "Digikey Part #" "1514-PN2222APBFREE-ND"
+			(at 247.65 91.44 0)
+			(hide yes)
+			(show_name no)
+			(do_not_autoplace no)
+			(effects
+				(font
+					(size 1.27 1.27)
+				)
 			)
 		)
