File: PCB/laser-tag-sao.kicad_pcb (KiCad board)
At the start: 2 copper layers, 99.8 x 43.6 mm, 18 parts, among them J1 SAO Connector, Q1 PN2222A, SW1 SW_Push, SW2 SW_Push, U1 ATTINY84A-PU, U2 TSOP38438, U3 OLED_0.91_128x32

Commit message: adding silkscreen
Parts:
- added G***: LOGO, LOGO, F.Cu at (208.1, 81.4)
Other:
- board text added: "Laser Tag SAO"
- board text added: "Made by Kai Pereira"

Commit message: cleaning up the ground fill a bit
Routing:
- net GND: track 5.92 -> 8.52 mm, vias 17 -> 24
Changed lines of the file:
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@@
+	)
+	(via
+		(at 202 69)
+		(size 0.6)
+		(drill 0.3)
+		(layers "F.Cu" "B.Cu")
+		(free yes)
+		(net "GND")
 	)
 	(via
@@
 	)
 	(via
+		(at 159 74.25)
+		(size 0.6)
+		(drill 0.3)
+		(layers "F.Cu" "B.Cu")
+		(free yes)
+		(net "GND")
+	)
+	(via
 		(at 212 70)
 		(size 0.6)
@@
 	)
 	(via
+		(at 163.25 76)
+		(size 0.6)
+		(drill 0.3)
+		(layers "F.Cu" "B.Cu")
+		(free yes)
+		(net "GND")
+	)
+	(via
 		(at 203 85)
 		(size 0.6)
@@
 	)
 	(via
+		(at 196 72.5)
+		(size 0.6)
+		(drill 0.3)
+		(layers "F.Cu" "B.Cu")
+		(free yes)
+		(net "GND")
+	)
+	(via
+		(at 189 71)
+		(size 0.6)
+		(drill 0.3)
+		(layers "F.Cu" "B.Cu")
+		(free yes)
+		(net "GND")
+	)
+	(via
 		(at 226.5 79.7)
 		(size 0.6)
@@
 	)
 	(via
+		(at 194 71)
+		(size 0.6)
+		(drill 0.3)
+		(layers "F.Cu" "B.Cu")
+		(free yes)
+		(net "GND")
+	)
+	(via
 		(at 214 77)
+		(size 0.6)
+		(drill 0.3)
+		(layers "F.Cu" "B.Cu")
+		(free yes)
+		(net "GND")
+	)
+	(via
+		(at 189.855751 77.348186)
 		(size 0.6)
 		(drill 0.3)
@@
 	)
 	(segment
+		(start 188 78.885)
+		(end 188 79)
+		(width 0.2)
+		(layer "B.Cu")
+		(net "GND")
+	)
+	(segment
+		(start 189.536814 77.348186)
+		(end 188 78.885)
+		(width 0.2)
+		(layer "B.Cu")
+		(net "GND")
+	)
+	(segment
 		(start 181.5 70)
 		(end 183 70)
@@
 		(width 0.2)
 		(layer "B.Cu")
+		(net "GND")
+	)
+	(segment
+		(start 189.855751 77.348186)
+		(end 189.536814 77.348186)
+		(width 0.2)
+		(layer "B.Cu")

Commit message: adding PCBWay branding
Other:
- board text added: "PCBWay"
Changed lines of the file:
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@@
+		)
+	)
+	(gr_text "PCBWay"
+		(at 195.75 72 0)
+		(layer "B.SilkS")
+		(effects
+			(font
+				(size 2 2)
+				(thickness 0.4)
+				(bold yes)
+			)
+			(justify left bottom mirror)
 		)
 	)

Commit message: new fab files
Other:
- board text removed: "PCBWay"
Changed lines of the file:
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@@
-		)
-	)
-	(gr_text "PCBWay"
-		(at 195.75 72 0)
-		(layer "B.SilkS")
-		(effects
-			(font
-				(size 2 2)
-				(thickness 0.4)
-				(bold yes)
-			)
-			(justify left bottom mirror)
 		)
 	)
